File: hardware/sync_and_burst.sch (KiCad schematic (older format))
At the start: 17 parts, among them SW2 SPDT_slide, U4 CD4013, U5 74HC4538, U6 LM1881, U7 74HC86

Commit message: add panel stuff
Parts:
- R12: value 1k (or 1.2k maybe) -> 1k
Changed lines of the file:
@@
 P 6900 1950
 F 0 "R12" V 6800 1950 50  0000 C CNN
-F 1 "1k (or 1.2k maybe)" V 7000 1950 50  0000 C CNN
+F 1 "1k" V 7000 1950 50  0000 C CNN
 F 2 "lib_fp:R_Axial_DIN0207_L6.3mm_D2.5mm_P7.62mm_Horizontal" V 6830 1950 50  0001 C CNN
 F 3 "~" H 6900 1950 50  0001 C CNN
