File: hardware/two_point_one_colorizer.sch (KiCad schematic (older format))
At the start: 34 parts, among them J1 Barrel_Jack, J2 rca, J3 mini-din4, J4 Conn_02x08_Odd_Even, J5 rca, Q1 2N3904, SW1 SPDT_slide, SW5 SW_DPDT_x2, U1 4069, U2 LM317, U3 CD4053, Y1 3.8MHZ_Crystal, Y2 4.4MHZ_Crystal

Commit message: add panel stuff
Connections:
- net video_in: no longer J3.4
- net at J2.1 (In), SW5.2 (B): now also J3.4
Changed lines of the file:
@@
 	1    0    0    -1
 $EndComp
-Wire Wire Line
-	1050 4750 1050 4100
-Connection ~ 1050 4100
-Wire Wire Line
-	1050 4100 1275 4100
 NoConn ~ 1250 5100
 $Comp
@@
 $EndComp
 Wire Wire Line
-	650  5100 650  4750
-Wire Wire Line
-	650  4750 1050 4750
-Wire Wire Line
 	650  5200 650  5550
 Wire Wire Line
@@
 Text GLabel 950  4100 0    50   Input ~ 0
 video_in
-Wire Wire Line
-	950  4100 1050 4100
 Text GLabel 2100 6700 2    50   Input ~ 0
 video_in
@@
 Text Notes 1000 6250 0    79   ~ 0
 SIGNAL_BYPASS
+Wire Wire Line
+	950  4100 1275 4100
+Wire Wire Line
+	650  5100 550  5100
+Wire Wire Line
+	550  5100 550  6600
+Wire Wire Line
+	550  6600 1350 6600
+Connection ~ 1350 6600
 $EndSCHEMATC
