File: hardware/colours.kicad_sch (KiCad schematic)
At the start: 27 parts, among them SW3 SPDT, SW4 SPDT, U10 74LS221, U7 74HC86, U9 74LS221

Commit message: getting ready to release
Parts:
- U10, U9: value 74LS221 -> 74LS123
