File: hardware/sync_and_burst.kicad_sch (KiCad schematic)
At the start: 17 parts, among them SW2 SPDT_slide, U4 CD4013, U5 74HC4538, U6 LM1881, U7 74HC86

Commit message: getting ready to release
Parts:
- R12: value 1k -> 680
