File: hardware/two_point_one_colorizer.kicad_pcb (KiCad board)
At the start: 2 copper layers, 100 x 100 mm, 93 parts, among them J1 Barrel_Jack, J2 rca, J3 mini-din4, J4 Conn_02x08_Odd_Even, J5 rca, Q1 2N3904, SW1 SPDT_slide, SW2 SPDT_slide, SW3 SPDT, SW4 SPDT, U1 4069, U10 74LS221, U2 LM317, U3 CD4053, U4 CD4013, U5 74HC4538, U6 LM1881, U7 74HC86, U8 LM393, U9 74LS221, Y1 3.8MHZ_Crystal, Y2 4.4MHZ_Crystal

Commit message: add panel stuff
Parts:
- removed J4: Conn_02x08_Odd_Even, Connector_PinHeader_2.54mm:PinHeader_2x08_P2.54mm_Vertical
- removed R21, R22: 10k, lib_fp:R_Axial_DIN0207_L6.3mm_D2.5mm_P7.62mm_Horizontal
- removed the REF** at (201.5, 38.5)
- removed the REF** at (201.5, 131.5)
- removed the REF** at (108.5, 131.5)
- removed the REF** at (108.5, 38.6)
- added REF**: MountingHole_3.2mm_M3, MountingHole:MountingHole_3.2mm_M3, F.Cu at (108.6, 38.5)
- added REF**: MountingHole_3.2mm_M3, MountingHole:MountingHole_3.2mm_M3, F.Cu at (201.7, 38.5)
- added REF**: MountingHole_3.2mm_M3, MountingHole:MountingHole_3.2mm_M3, F.Cu at (201.6, 131.5)
- added REF**: MountingHole_3.2mm_M3, MountingHole:MountingHole_3.2mm_M3, F.Cu at (108.5, 131.5)
- added SW5: SW_DPDT_x2, lib_fp:dpdt_mini_toggle_switch_tayda, F.Cu at (138.2, 32.4)
- R12: value 1k (or 1.2k maybe) -> 1k
- R17, R18: value 22k -> 18k
- R19, R20: value 82k -> 22k
- RV8, RV9: footprint lib_fp:Pot_trim_3362_tayda -> lib_fp:Potentiometer_Vertical_Large
- moved C4 28.4 mm to (172.5, 38.3)
- moved R30 23.3 mm to (106.6, 125.8)
- moved U2 22.7 mm to (162.7, 38.5)
- moved J3 21.8 mm to (113.9, 60.5)
- moved R1 17.6 mm to (131.6, 49.8)
- moved SW4 17.5 mm to (140.8, 127.5), turned to -90 degrees
- moved C20 14.8 mm to (153.1, 111.7)
- moved R17 13.4 mm to (169.8, 80.8), turned to 0 degrees
- moved R18 13.0 mm to (107.0, 80.9), turned to 0 degrees
- moved R19 12.9 mm to (177.4, 84.4), turned to 180 degrees
- moved R4 12.5 mm to (109.9, 69.6), turned to -90 degrees
- moved R20 10.6 mm to (107.0, 84.6)
- moved RV8 10.3 mm to (190.4, 133.4), turned to 90 degrees
- moved RV9 10.2 mm to (125.3, 133.4), turned to 90 degrees
- moved R32 9.49 mm to (139.1, 125.6)
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Connections:
- C2 pad 2: Net-(C2-Pad2) -> video_in
- J2 pad 1: Net-(C2-Pad2) -> Net-(J2-Pad1)
- J3 pad 3: Net-(J3-Pad3) -> unconnected-(J3-Pad3)
- J3 pad 4: Net-(C2-Pad2) -> Net-(J2-Pad1)
- R1 pad 1: Net-(C2-Pad2) -> video_in
- R17 pad 1: Net-(C16-Pad1) -> GND
- R18 pad 1: Net-(C17-Pad1) -> GND
- R19 pad 2: Net-(C16-Pad1) -> Net-(R19-Pad2)
- R20 pad 2: Net-(C17-Pad1) -> Net-(R20-Pad2)
- R8 pad 1: Net-(J5-Pad1) -> video_out
- RV1 pad 3: Net-(RV1-Pad3) -> unconnected-(RV1-Pad3)
- RV2 pad 1: +5V -> Net-(R19-Pad2)
- RV2 pad 2: Net-(R17-Pad2) -> Net-(C16-Pad1)
- RV2 pad 3: GND -> Net-(R17-Pad2)
- RV3 pad 1: +5V -> Net-(R20-Pad2)
- RV3 pad 2: Net-(R18-Pad2) -> Net-(C17-Pad1)
- RV3 pad 3: GND -> Net-(R18-Pad2)
- RV4 pad 3: Net-(RV4-Pad3) -> unconnected-(RV4-Pad3)
- RV5 pad 3: Net-(RV5-Pad3) -> unconnected-(RV5-Pad3)
- RV6 pad 3: Net-(RV6-Pad3) -> unconnected-(RV6-Pad3)
- RV7 pad 3: Net-(RV7-Pad3) -> unconnected-(RV7-Pad3)
- RV8 pad 3: Net-(RV8-Pad3) -> unconnected-(RV8-Pad3)
- RV9 pad 3: Net-(RV9-Pad3) -> unconnected-(RV9-Pad3)
- SW3 pad 3: Net-(SW3-Pad3) -> unconnected-(SW3-Pad3)
- SW4 pad 3: Net-(SW4-Pad3) -> unconnected-(SW4-Pad3)
- U1 pad 10: Net-(U1-Pad10) -> unconnected-(U1-Pad10)
- U1 pad 11: Net-(U1-Pad11) -> unconnected-(U1-Pad11)
- U1 pad 12: Net-(U1-Pad12) -> unconnected-(U1-Pad12)
- U1 pad 13: Net-(U1-Pad13) -> unconnected-(U1-Pad13)
- U1 pad 5: Net-(U1-Pad5) -> unconnected-(U1-Pad5)
- U1 pad 6: Net-(U1-Pad6) -> unconnected-(U1-Pad6)
- U1 pad 8: Net-(U1-Pad8) -> unconnected-(U1-Pad8)
- U1 pad 9: Net-(U1-Pad9) -> unconnected-(U1-Pad9)
- U10 pad 12: Net-(U10-Pad12) -> unconnected-(U10-Pad12)
- U10 pad 13: Net-(U10-Pad13) -> unconnected-(U10-Pad13)
- U4 pad 10: Net-(U4-Pad10) -> unconnected-(U4-Pad10)
- U4 pad 11: Net-(U4-Pad11) -> unconnected-(U4-Pad11)
- U4 pad 12: Net-(U4-Pad12) -> unconnected-(U4-Pad12)
- U4 pad 13: Net-(U4-Pad13) -> unconnected-(U4-Pad13)
- U4 pad 8: Net-(U4-Pad8) -> unconnected-(U4-Pad8)
- U4 pad 9: Net-(U4-Pad9) -> unconnected-(U4-Pad9)
- U5 pad 10: Net-(U5-Pad10) -> unconnected-(U5-Pad10)
- U5 pad 11: Net-(U5-Pad11) -> unconnected-(U5-Pad11)
- U5 pad 12: Net-(U5-Pad12) -> unconnected-(U5-Pad12)
- U5 pad 13: Net-(U5-Pad13) -> unconnected-(U5-Pad13)
- U5 pad 14: Net-(U5-Pad14) -> unconnected-(U5-Pad14)
- U5 pad 15: Net-(U5-Pad15) -> unconnected-(U5-Pad15)
- U5 pad 5: Net-(R10-Pad2) -> Net-(U5-Pad5)
- U5 pad 6: Net-(U5-Pad6) -> unconnected-(U5-Pad6)
- U5 pad 9: Net-(U5-Pad9) -> unconnected-(U5-Pad9)
- U6 pad 3: Net-(U6-Pad3) -> unconnected-(U6-Pad3)
- U6 pad 5: Net-(U6-Pad5) -> Net-(U5-Pad5)
- U6 pad 7: Net-(U6-Pad7) -> unconnected-(U6-Pad7)
- U7 pad 11: Net-(U7-Pad11) -> unconnected-(U7-Pad11)
- U7 pad 12: Net-(U7-Pad12) -> unconnected-(U7-Pad12)
- U7 pad 13: Net-(U7-Pad13) -> unconnected-(U7-Pad13)
- U9 pad 12: Net-(U9-Pad12) -> unconnected-(U9-Pad12)
- U9 pad 13: Net-(U9-Pad13) -> unconnected-(U9-Pad13)
Routing:
- net Net-(U5-Pad5): track 0.00 -> 57.0 mm, vias 0 -> 1
- net video_out: track 0.00 -> 55.6 mm, vias 0 -> 1
- net Net-(J5-Pad1): track 10.1 -> 63.7 mm, vias 0 -> 1
- net Net-(J2-Pad1): track 0.00 -> 45.8 mm
- net GND: track 40.5 -> 85.0 mm, vias 2 -> 6
- net video_in: track 0.00 -> 34.9 mm
- net Net-(R10-Pad2): track 153.8 -> 122.5 mm, vias 1 -> 0
- net Net-(C2-Pad2): track 30.6 -> 0.00 mm
- net Net-(C21-Pad1): track 16.6 -> 42.4 mm
- net Net-(U6-Pad5): track 25.4 -> 0.00 mm
- net Net-(R30-Pad1): track 5.23 -> 30.3 mm
- net unconnected-(U6-Pad3): track 0.00 -> 25.0 mm
- net Net-(U6-Pad3): track 25.0 -> 0.00 mm
- net 1.25v: track 219.7 -> 242.4 mm
- net Net-(R19-Pad2): track 0.00 -> 21.6 mm
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Other:
- net class Default removed
- board text added: "_^ 09"
- board text added: "two_point_one_colorizer v0_4_1 based on rob schafer design updated by cyberboy666"
- board text removed: "_^ XX"
- board text removed: "two_point_one_colorizer v0_3 based on rob schafer design updated by cyberboy666"

Commit message: getting ready to release
Parts:
- removed J3: mini-din4, lib_fp:mini-din-4-vertical_KMDVLX-4S-N-1
- C14: value 0.1n -> 100p
- R12: value 1k -> 680
- RV8, RV9: value 5k_trim -> 5k_pot
- U1: value 4069 -> CD4069
- U10, U9: value 74LS221 -> 74LS123
- Y1: value 3.8MHZ_Crystal -> 3.57Mhz_crystal
- Y2: value 4.4MHZ_Crystal -> 4.43Mhz_crystal
- moved R5 2.66 mm to (141.5, 48.8)
Routing:
- net /colours/colour1: track 280.6 -> 257.6 mm
- net Net-(J2-In): track 45.8 -> 31.3 mm
Other:
- board text added: "-> bypass"
- board text added: "JLCJLCJLCJLC"
- board text added: "phase alternating on/off"
- board text added: "two_point_one_colorizer v1_0_0 based on rob schafer design updated by cyberboy666"
- board text removed: "two_point_one_colorizer v0_4_1 based on rob schafer design updated by cyberboy666"
