File: panel/default_panel/default_panel.kicad_pcb (KiCad board)
At the start: 2 copper layers, 100 x 100 mm, 0 parts

Commit message: getting ready to release
Other:
- outline, holes or cut-outs redrawn
- board text added: "default panel two_point_one_colorizer v1_0_0 based on rob schafer design updated by cyberboy666"
- board text removed: "default panel mk_i for two_point_one_colorizer v0_4_1 based on rob schafer design updated by cyberboy666"
Changed lines of the file:
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@@
-(kicad_pcb (version 20211014) (generator pcbnew)
+(kicad_pcb (version 20221018) (generator pcbnew)
   (general
     (thickness 1.6)
@@
     (pcbplotparams
       (layerselection 0x00010fc_ffffffff)
+      (plot_on_all_layers_selection 0x0000000_00000000)
       (disableapertmacros false)
       (usegerberextensions false)
@@
       (usegerberadvancedattributes true)
       (creategerberjobfile true)
-      (svguseinch false)
+      (dashed_line_dash_ratio 12.000000)
+      (dashed_line_gap_ratio 3.000000)
       (svgprecision 6)
-      (excludeedgelayer true)
       (plotframeref false)
       (viasonmask false)
@@
   )
   (net 0 "")
-  (gr_line (start 88.55 136.5) (end 86.65 134.3) (layer "F.SilkS") (width 0.35))
-  (gr_line (start 96.75 82.575) (end 93.05 85.825) (layer "F.SilkS") (width 0.35))
-  (gr_line (start 96.4 75.1) (end 93.15 71.4) (layer "F.SilkS") (width 0.35))
-  (gr_line (start 137.4 137) (end 139.7 133.8) (layer "F.SilkS") (width 0.35))
-  (gr_line (start 144.3 98.1) (end 144.3 123.7) (layer "F.SilkS") (width 0.35))
-  (gr_line (start 130.1 85.85) (end 126.4 82.6) (layer "F.SilkS") (width 0.35))
-  (gr_line (start 81.1 98.2) (end 81.1 123.8) (layer "F.SilkS") (width 0.35))
-  (gr_line (start 129.45 71.35) (end 126.2 75.05) (layer "F.SilkS") (width 0.35))
-  (gr_circle (center 91.6 140.4) (end 95.6 140.4) (layer "Edge.Cuts") (width 0.1) (fill none))
-  (gr_line (start 62.7 48) (end 162.7 48) (layer "Edge.Cuts") (width 0.15))
-  (gr_circle (center 135.8 124.3) (end 139.8 124.3) (layer "Edge.Cuts") (width 0.1) (fill none))
-  (gr_circle (center 70.2 124.8) (end 74.2 124.8) (layer "Edge.Cuts") (width 0.1) (fill none))
-  (gr_circle (center 112.7 138.9) (end 116.7 138.9) (layer "Edge.Cuts") (width 0.1) (fill none))
-  (gr_circle (center 66.2 144.5) (end 68 144.5) (layer "Edge.Cuts") (width 0.1) (fill none))
-  (gr_line (start 69.1 118.5) (end 62.7 118.5) (layer "Edge.Cuts") (width 0.1))
-  (gr_circle (center 145.6 138.9) (end 149.6 138.9) (layer "Edge.Cuts") (width 0.1) (fill none))
-  (gr_circle (center 155.4 124.3) (end 159.4 124.3) (layer "Edge.Cuts") (width 0.1) (fill none))
-  (gr_circle (center 134.2 140.7) (end 138.2 140.7) (layer "Edge.Cuts") (width 0.1) (fill none))
-  (gr_line (start 62.7 105.2) (end 69.1 105.2) (layer "Edge.Cuts") (width 0.1))
-  (gr_line (start 156.95 118.4) (end 156.95 105.1) (layer "Edge.Cuts") (width 0.1))
-  (gr_circle (center 80.9 87) (end 84.9 87) (layer "Edge.Cuts") (width 0.1) (fill none))
-  (gr_line (start 62.7 148) (end 62.7 118.5) (layer "Edge.Cuts") (width 0.15))
-  (gr_circle (center 80.5 138.9) (end 84.5 138.9) (layer "Edge.Cuts") (width 0.1) (fill none))
-  (gr_line (start 162.7 48) (end 162.7 105.1) (layer "Edge.Cuts") (width 0.15))
-  (gr_line (start 162.7 118.4) (end 162.7 148) (layer "Edge.Cuts") (width 0.15))
-  (gr_circle (center 159.2 144.5) (end 161 144.5) (layer "Edge.Cuts") (width 0.1) (fill none))
-  (gr_circle (center 91.1 124.8) (end 95.1 124.8) (layer "Edge.Cuts") (width 0.1) (fill none))
-  (gr_line (start 69.1 105.2) (end 69.1 118.5) (layer "Edge.Cuts") (width 0.1))
-  (gr_line (start 156.95 105.1) (end 162.7 105.1) (layer "Edge.Cuts") (width 0.1))
-  (gr_line (start 162.7 148) (end 62.7 148) (layer "Edge.Cuts") (width 0.15))
-  (gr_line (start 162.7 118.4) (end 156.95 118.4) (layer "Edge.Cuts") (width 0.1))
-  (gr_line (start 62.7 105.2) (end 62.7 48) (layer "Edge.Cuts") (width 0.15))
-  (gr_circle (center 159.2 51.5) (end 161 51.5) (layer "Edge.Cuts") (width 0.1) (fill none))
-  (gr_circle (center 144.4 86.7) (end 148.4 86.7) (layer "Edge.Cuts") (width 0.1) (fill none))
-  (gr_circle (center 95.9 54.8) (end 99.9 54.8) (layer "Edge.Cuts") (width 0.1) (fill none))
-  (gr_circle (center 66.2 51.5) (end 68 51.5) (layer "Edge.Cuts") (width 0.1) (fill none))
-  (gr_circle (center 69.7 59.4) (end 76.2 59.4) (layer "Edge.Cuts") (width 0.1) (fill none))
-  (gr_circle (center 155.7 59.5) (end 162.2 59.5) (layer "Edge.Cuts") (width 0.1) (fill none))
+  (gr_line (start 88.55 136.5) (end 86.65 134.3)
+    (stroke (width 0.35) (type solid)) (layer "F.SilkS"))
+  (gr_line (start 96.75 82.575) (end 93.05 85.825)
+    (stroke (width 0.35) (type solid)) (layer "F.SilkS"))
+  (gr_line (start 96.4 75.1) (end 93.15 71.4)
+    (stroke (width 0.35) (type solid)) (layer "F.SilkS"))
+  (gr_line (start 137.4 137) (end 139.7 133.8)
+    (stroke (width 0.35) (type solid)) (layer "F.SilkS"))
+  (gr_line (start 144.3 98.1) (end 144.3 123.7)
+    (stroke (width 0.35) (type solid)) (layer "F.SilkS"))
+  (gr_line (start 130.1 85.85) (end 126.4 82.6)
+    (stroke (width 0.35) (type solid)) (layer "F.SilkS"))
+  (gr_line (start 81.1 98.2) (end 81.1 123.8)
+    (stroke (width 0.35) (type solid)) (layer "F.SilkS"))
+  (gr_line (start 129.45 71.35) (end 126.2 75.05)
+    (stroke (width 0.35) (type solid)) (layer "F.SilkS"))
+  (gr_circle (center 91.6 140.4) (end 95.6 140.4)
+    (stroke (width 0.1) (type solid)) (fill none) (layer "Edge.Cuts"))
+  (gr_line (start 62.7 48) (end 162.7 48)
+    (stroke (width 0.15) (type solid)) (layer "Edge.Cuts"))
+  (gr_circle (center 135.8 124.3) (end 139.8 124.3)
+    (stroke (width 0.1) (type solid)) (fill none) (layer "Edge.Cuts"))
+  (gr_circle (center 70.2 124.8) (end 74.2 124.8)
+    (stroke (width 0.1) (type solid)) (fill none) (layer "Edge.Cuts"))
+  (gr_circle (center 112.7 138.9) (end 116.7 138.9)
+    (stroke (width 0.1) (type solid)) (fill none) (layer "Edge.Cuts"))
+  (gr_circle (center 66.2 144.5) (end 68 144.5)
+    (stroke (width 0.1) (type solid)) (fill none) (layer "Edge.Cuts"))
+  (gr_line (start 69.1 118.5) (end 62.7 118.5)
+    (stroke (width 0.1) (type solid)) (layer "Edge.Cuts"))
+  (gr_circle (center 145.6 138.9) (end 149.6 138.9)
+    (stroke (width 0.1) (type solid)) (fill none) (layer "Edge.Cuts"))
+  (gr_circle (center 155.4 124.3) (end 159.4 124.3)
+    (stroke (width 0.1) (type solid)) (fill none) (layer "Edge.Cuts"))
+  (gr_circle (center 134.2 140.7) (end 138.2 140.7)
+    (stroke (width 0.1) (type solid)) (fill none) (layer "Edge.Cuts"))
+  (gr_line (start 62.7 105.2) (end 69.1 105.2)
+    (stroke (width 0.1) (type solid)) (layer "Edge.Cuts"))
+  (gr_line (start 156.95 118.4) (end 156.95 105.1)
+    (stroke (width 0.1) (type solid)) (layer "Edge.Cuts"))
+  (gr_circle (center 80.9 87) (end 84.9 87)
+    (stroke (width 0.1) (type solid)) (fill none) (layer "Edge.Cuts"))
+  (gr_line (start 62.7 148) (end 62.7 118.5)
+    (stroke (width 0.15) (type solid)) (layer "Edge.Cuts"))
+  (gr_circle (center 80.5 138.9) (end 84.5 138.9)
+    (stroke (width 0.1) (type solid)) (fill none) (layer "Edge.Cuts"))
+  (gr_line (start 162.7 48) (end 162.7 105.1)
+    (stroke (width 0.15) (type solid)) (layer "Edge.Cuts"))
+  (gr_line (start 162.7 118.4) (end 162.7 148)
+    (stroke (width 0.15) (type solid)) (layer "Edge.Cuts"))
+  (gr_circle (center 159.2 144.5) (end 161 144.5)
+    (stroke (width 0.1) (type solid)) (fill none) (layer "Edge.Cuts"))
+  (gr_circle (center 91.1 124.8) (end 95.1 124.8)
+    (stroke (width 0.1) (type solid)) (fill none) (layer "Edge.Cuts"))
+  (gr_line (start 69.1 105.2) (end 69.1 118.5)
+    (stroke (width 0.1) (type solid)) (layer "Edge.Cuts"))
+  (gr_line (start 156.95 105.1) (end 162.7 105.1)
+    (stroke (width 0.1) (type solid)) (layer "Edge.Cuts"))
+  (gr_line (start 162.7 148) (end 62.7 148)
+    (stroke (width 0.15) (type solid)) (layer "Edge.Cuts"))
+  (gr_line (start 162.7 118.4) (end 156.95 118.4)
+    (stroke (width 0.1) (type solid)) (layer "Edge.Cuts"))
+  (gr_line (start 62.7 105.2) (end 62.7 48)
+    (stroke (width 0.15) (type solid)) (layer "Edge.Cuts"))
+  (gr_circle (center 159.2 51.5) (end 161 51.5)
+    (stroke (width 0.1) (type solid)) (fill none) (layer "Edge.Cuts"))
+  (gr_circle (center 144.4 86.7) (end 148.4 86.7)
+    (stroke (width 0.1) (type solid)) (fill none) (layer "Edge.Cuts"))
+  (gr_circle (center 95.9 54.8) (end 99.9 54.8)
+    (stroke (width 0.1) (type solid)) (fill none) (layer "Edge.Cuts"))
+  (gr_circle (center 66.2 51.5) (end 68 51.5)
+    (stroke (width 0.1) (type solid)) (fill none) (layer "Edge.Cuts"))
+  (gr_circle (center 155.7 59.5) (end 162.2 59.5)
+    (stroke (width 0.1) (type solid)) (fill none) (layer "Edge.Cuts"))
   (gr_text "_^ 09" (at 140.8 72.35) (layer "B.SilkS")
     (effects (font (size 5 5) (thickness 0.6)) (justify mirror))
   )
-  (gr_text "default panel mk_i for\ntwo_point_one_colorizer  v0_4_1\nbased on rob schafer design\nupdated by cyberboy666" (at 158 70.5 90) (layer "B.SilkS")
+  (gr_text "default panel\ntwo_point_one_colorizer  v1_0_0\nbased on rob schafer design\nupdated by cyberboy666" (at 158 70.5 90) (layer "B.SilkS")
     (effects (font (size 1.2 1.2) (thickness 0.2)) (justify left mirror))
   )
