File: panel/default_panel/default_panel.kicad_pcb (KiCad board)
At the start: 2 copper layers, 100 x 100 mm, 0 parts

Commit message: update panels
Other:
- outline, holes or cut-outs redrawn
- board text added: "JLCJLCJLCJLC"
Changed lines of the file:
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@@
   (gr_line (start 129.45 71.35) (end 126.2 75.05)
     (stroke (width 0.35) (type solid)) (layer "F.SilkS"))
+  (gr_circle (center 69.6 59.45) (end 76.1 59.45)
+    (stroke (width 0.1) (type solid)) (fill none) (layer "Edge.Cuts"))
   (gr_circle (center 91.6 140.4) (end 95.6 140.4)
     (stroke (width 0.1) (type solid)) (fill none) (layer "Edge.Cuts"))
@@
   (gr_circle (center 66.2 51.5) (end 68 51.5)
     (stroke (width 0.1) (type solid)) (fill none) (layer "Edge.Cuts"))
-  (gr_circle (center 155.7 59.5) (end 162.2 59.5)
+  (gr_circle (center 155.7 59.45) (end 162.2 59.45)
     (stroke (width 0.1) (type solid)) (fill none) (layer "Edge.Cuts"))
   (gr_text "_^ 09" (at 140.8 72.35) (layer "B.SilkS")
@@
     (effects (font (size 1.5 1.5) (thickness 0.3)) (justify mirror))
   )
+  (gr_text "JLCJLCJLCJLC" (at 157.35 147.15) (layer "B.SilkS")
+    (effects (font (size 1 1) (thickness 0.15)) (justify mirror))
+  )
   (gr_text "COLOR_TWO" (at 144.3 131.2) (layer "F.SilkS")
