File: panel/eurorack_panel/eurorack_panel.kicad_pcb (KiCad board)
At the start: 2 copper layers, 101.7 x 128.6 mm, 0 parts

Commit message: getting ready to release
Other:
- outline, holes or cut-outs redrawn
- board text added: "eurorack_panel two_point_one_colorizer v1_0_0 based on rob schafer design updated by cyberboy666"
- board text removed: "eurorack_panel mk_i for two_point_one_colorizer v0_4_1 based on rob schafer design updated by cyberboy666"
