File: panel/eurorack_panel/eurorack_panel.kicad_pcb (KiCad board)
At the start: 2 copper layers, 101.7 x 128.6 mm, 0 parts

Commit message: update panels
Other:
- outline, holes or cut-outs redrawn
Changed lines of the file:
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@@
   (gr_line (start 69.1 105.2) (end 69.1 118.5)
     (stroke (width 0.1) (type solid)) (layer "Edge.Cuts"))
+  (gr_circle (center 69.7 59.5) (end 63.2 59.5)
+    (stroke (width 0.1) (type solid)) (fill none) (layer "Edge.Cuts"))
   (gr_line (start 61.8 105.2) (end 69.1 105.2)
     (stroke (width 0.1) (type solid)) (layer "Edge.Cuts"))
